Commit message: update

File: src/isaac_ros_nvblox/nvblox_examples/nvblox_examples_bringup/config/urdf/2_realsense_go2_camera0_base.urdf.xacro (robot description, xacro)
@@ -31,5 +31,5 @@
     <parent link="sensor_head_link"/>
     <child link="base_link"/>
-    <origin xyz="-0.3284235 0 -0.0942744" rpy="0 0 0"/>
+    <origin xyz="-0.3384235 0 -0.0792744" rpy="0 0 0"/>
   </joint>
   <link name="base_link"/>
